Commit message: 20230320_수정

File: patrol_scout_mini/scout_description/urdf/mini.xacro (robot description, xacro)
@@ -14,4 +14,12 @@
     <xacro:property name="base_y_size" value="0.3816" />
     <xacro:property name="base_z_size" value="0.10357" />
+    <xacro:property name="hokuyo_size" value="0.05" />
+    <!-- Main body radius and height -->
+    <!-- Main Body Cylinder base   -->
+    <xacro:property name="base_height" value="0.02" />
+    <xacro:property name="base_radius" value="0.15" />
+    <xacro:property name="base_mass" value="5.0" /> <!-- in kg-->
+    <!-- <xacro:property name="hokuyo_size" value="5.0" /> -->
+    <xacro:property name="hokuyo_size" value="0.05" />
     <xacro:property name="wheelbase" value="0.463951"/>
     <xacro:property name="track" value="0.416503"/>
@@ -112,3 +120,65 @@
     <!-- Gazebo definitions  -->
     <xacro:include filename="$(find scout_description)/urdf/scout_mini.gazebo" />
+    <!-- <joint name="laser" type="fixed">
+    <origin xyz="-0.005 0.00 0.43" rpy="3.14159 0 0" />
+    <parent link="base_link" />
+    <child link="base_laser_link" />
+    </joint> -->
+    <!-- <link name="base_laser_link">
+      <visual>
+        <geometry>
+          <box size="0.06 0.06 0.06" />
+        </geometry>
+        <material name="Green" />
+      </visual>
+      <inertial>
+        <mass value="0.000001" />
+        <origin xyz="0 0 0" />
+        <inertia ixx="0.0001" ixy="0.0" ixz="0.0"
+          iyy="0.0001" iyz="0.0"
+          izz="0.0001" />
+      </inertial>
+    </link> -->
+    <!-- <link name="laser_link">
+    <visual>
+      <origin xyz="0 0 0" rpy="0 0 0" />
+      <geometry>
+        <box size="${hokuyo_size} ${hokuyo_size} ${hokuyo_size}"/>
+      </geometry>
+      <material name="Blue" />
+    </visual>
+    </link>
+    <joint name="hokuyo_joint" type="fixed">
+      <origin xyz="${base_radius - hokuyo_size/2} 0 ${base_height+hokuyo_size/4}" rpy="0 0 0" />
+      <parent link="base_link"/>
+      <child link="laser_link" />
+    </joint>
+    <gazebo reference="laser_link">
+        <material>Gazebo/Blue</material>
+        <turnGravityOff>false</turnGravityOff>
+        <sensor type="ray" name="head_hokuyo_sensor">
+          <pose>${hokuyo_size/2} 0 0 0 0 0</pose>
+          <visualize>true</visualize>
+          <update_rate>40</update_rate>
+          <ray>
+            <scan>
+              <horizontal>
+                <samples>720</samples>
+                <resolution>1</resolution>
+                <min_angle>-1.570796</min_angle>
+                <max_angle>1.570796</max_angle>
+              </horizontal>
+            </scan>
+            <range>
+              <min>0.10</min>
+              <max>10.0</max>
+              <resolution>0.001</resolution>
+            </range>
+          </ray>
+          <plugin name="gazebo_ros_head_hokuyo_controller" filename="libgazebo_ros_laser.so">
+            <topicName>/scan</topicName>
+            <frameName>laser_link</frameName>
+          </plugin>
+        </sensor>
+    </gazebo> -->
 </robot>
